File: Conversor/Proyecto-KiCAD/Proyecto-KiCAD.kicad_sch (KiCad schematic)
At the start: 0 parts

Commit message: Importar esquematicos y PCBs de referencia a KiCAD
Parts:
- added Q1, Q2, Q3, Q4: (no value), symbol Componentes proyecto:IRFP150
- added U1, U2: (no value), symbol Componentes proyecto:UCC21540
Connections:
- new net: Q1.3 (S), Q2.1 (D), U1.14 (VSSA)
- new net: Q2.2 (G), U1.10 (OUTB)
- new net: Q2.3 (S), Q4.3 (S), U1.9 (VSSB), U2.9 (VSSB)
- new net: Q1.2 (G), U1.15 (OUTA)
- new net: Q4.2 (G), U2.10 (OUTB)
- new net: Q3.3 (S), Q4.1 (D), U2.14 (VSSA)
- new net: Q3.2 (G), U2.15 (OUTA)
- new net: Q1.1 (D), Q3.1 (D)
Changed lines of the file:
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@@
 (kicad_sch (version 20211123) (generator eeschema)
   (paper "A4")
+  (junction (at 180.34 100.33) (diameter 0) (color 0 0 0 0)
+  )
+  (junction (at 124.46 99.06) (diameter 0) (color 0 0 0 0)
+  )
+  (junction (at 180.34 82.55) (diameter 0) (color 0 0 0 0)
+  )
+  (junction (at 124.46 81.28) (diameter 0) (color 0 0 0 0)
+  )
+  (wire (pts (xy 113.03 99.06) (xy 124.46 99.06))
+    (stroke (width 0) (type default) (color 0 0 0 0))
+  )
+  (wire (pts (xy 165.1 92.71) (xy 165.1 100.33))
+    (stroke (width 0) (type default) (color 0 0 0 0))
+  )
+  (wire (pts (xy 172.72 90.17) (xy 172.72 93.98))
+    (stroke (width 0) (type default) (color 0 0 0 0))
+  )
+  (wire (pts (xy 113.03 91.44) (xy 113.03 99.06))
+    (stroke (width 0) (type default) (color 0 0 0 0))
+  )
+  (wire (pts (xy 180.34 100.33) (xy 180.34 99.06))
+    (stroke (width 0) (type default) (color 0 0 0 0))
+  )
+  (wire (pts (xy 180.34 81.28) (xy 180.34 82.55))
+    (stroke (width 0) (type default) (color 0 0 0 0))
+  )
+  (wire (pts (xy 106.68 78.74) (xy 116.84 78.74))
+    (stroke (width 0) (type default) (color 0 0 0 0))
+  )
+  (wire (pts (xy 180.34 82.55) (xy 180.34 88.9))
+    (stroke (width 0) (type default) (color 0 0 0 0))
+  )
+  (wire (pts (xy 165.1 90.17) (xy 172.72 90.17))
+    (stroke (width 0) (type default) (color 0 0 0 0))
+  )
+  (wire (pts (xy 172.72 80.01) (xy 172.72 76.2))
+    (stroke (width 0) (type default) (color 0 0 0 0))
+  )
+  (wire (pts (xy 106.68 88.9) (xy 116.84 88.9))
+    (stroke (width 0) (type default) (color 0 0 0 0))
+  )
+  (wire (pts (xy 124.46 80.01) (xy 124.46 81.28))
+    (stroke (width 0) (type default) (color 0 0 0 0))
+  )
+  (wire (pts (xy 124.46 105.41) (xy 180.34 105.41))
+    (stroke (width 0) (type default) (color 0 0 0 0))
+  )
+  (wire (pts (xy 116.84 88.9) (xy 116.84 92.71))
+    (stroke (width 0) (type default) (color 0 0 0 0))
+  )
+  (wire (pts (xy 106.68 81.28) (xy 124.46 81.28))
+    (stroke (width 0) (type default) (color 0 0 0 0))
+  )
+  (wire (pts (xy 180.34 64.77) (xy 124.46 64.77))
+    (stroke (width 0) (type default) (color 0 0 0 0))
+  )
+  (wire (pts (xy 106.68 91.44) (xy 113.03 91.44))
+    (stroke (width 0) (type default) (color 0 0 0 0))
+  )
+  (wire (pts (xy 124.46 97.79) (xy 124.46 99.06))
+    (stroke (width 0) (type default) (color 0 0 0 0))
+  )
+  (wire (pts (xy 124.46 64.77) (xy 124.46 69.85))
+    (stroke (width 0) (type default) (color 0 0 0 0))
+  )
+  (wire (pts (xy 180.34 105.41) (xy 180.34 100.33))
+    (stroke (width 0) (type default) (color 0 0 0 0))
+  )
+  (wire (pts (xy 124.46 99.06) (xy 124.46 105.41))
+    (stroke (width 0) (type default) (color 0 0 0 0))
+  )
+  (wire (pts (xy 165.1 82.55) (xy 180.34 82.55))
+    (stroke (width 0) (type default) (color 0 0 0 0))
+  )
+  (wire (pts (xy 124.46 81.28) (xy 124.46 87.63))
+    (stroke (width 0) (type default) (color 0 0 0 0))
+  )
+  (wire (pts (xy 165.1 100.33) (xy 180.34 100.33))
+    (stroke (width 0) (type default) (color 0 0 0 0))
+  )
+  (wire (pts (xy 116.84 78.74) (xy 116.84 74.93))
+    (stroke (width 0) (type default) (color 0 0 0 0))
+  )
+  (wire (pts (xy 180.34 71.12) (xy 180.34 64.77))
+    (stroke (width 0) (type default) (color 0 0 0 0))
+  )
+  (wire (pts (xy 165.1 80.01) (xy 172.72 80.01))
+    (stroke (width 0) (type default) (color 0 0 0 0))
+  )
+  (symbol (lib_id "Componentes proyecto:IRFP150") (at 124.46 91.44 0) (unit 1)
+    (in_bom yes) (on_board yes)
+    (property "Reference" "Q2" (id 0) (at 128.27 92.7099 0)
+      (effects (font (size 1.27 1.27)) (justify left))
+    )
+    (property "Value" "" (id 1) (at 128.27 95.2499 0)
+      (effects (font (size 1.27 1.27)) (justify left))
+    )
+    (property "Footprint" "" (id 2) (at 124.46 91.44 0)
+      (effects (font (size 1.27 1.27)) hide)
+    )
+    (property "Datasheet" "" (id 3) (at 124.46 91.44 0)
+      (effects (font (size 1.27 1.27)) hide)
+    )
+    (pin "1")
+    (pin "2")
+    (pin "3")
+  )
+  (symbol (lib_id "Componentes proyecto:UCC21540") (at 95.25 83.82 0) (unit 1)
+    (in_bom yes) (on_board yes) (fields_autoplaced)
+    (property "Reference" "U1" (id 0) (at 95.25 68.58 0))
+    (property "Value" "" (id 1) (at 95.25 71.12 0))
+    (property "Footprint" "" (id 2) (at 95.25 82.55 0)
+      (effects (font (size 1.27 1.27)) hide)
+    )
+    (property "Datasheet" "" (id 3) (at 95.25 82.55 0)
+      (effects (font (size 1.27 1.27)) hide)
+    )
+    (pin "1")
+    (pin "10")
+    (pin "11")
+    (pin "14")
+    (pin "15")
+    (pin "16")
+    (pin "2")
+    (pin "3")
+    (pin "4")
+    (pin "5")
+    (pin "6")
+    (pin "8")
+    (pin "9")
+  )
+  (symbol (lib_id "Componentes proyecto:UCC21540") (at 153.67 85.09 0) (unit 1)
+    (in_bom yes) (on_board yes) (fields_autoplaced)
+    (property "Reference" "U2" (id 0) (at 153.67 69.85 0))
+    (property "Value" "" (id 1) (at 153.67 72.39 0))
+    (property "Footprint" "" (id 2) (at 153.67 83.82 0)
+      (effects (font (size 1.27 1.27)) hide)
+    )
+    (property "Datasheet" "" (id 3) (at 153.67 83.82 0)
+      (effects (font (size 1.27 1.27)) hide)
+    )
+    (pin "1")
+    (pin "10")
+    (pin "11")
+    (pin "14")
+    (pin "15")
+    (pin "16")
+    (pin "2")
+    (pin "3")
+    (pin "4")
+    (pin "5")
+    (pin "6")
+    (pin "8")
+    (pin "9")
+  )
+  (symbol (lib_id "Componentes proyecto:IRFP150") (at 180.34 74.93 0) (unit 1)
+    (in_bom yes) (on_board yes) (fields_autoplaced)
+    (property "Reference" "Q3" (id 0) (at 184.15 74.9299 0)
+      (effects (font (size 1.27 1.27)) (justify left))
+    )
+    (property "Value" "" (id 1) (at 184.15 77.4699 0)
+      (effects (font (size 1.27 1.27)) (justify left))
+    )
+    (property "Footprint" "" (id 2) (at 180.34 74.93 0)
+      (effects (font (size 1.27 1.27)) hide)
+    )
+    (property "Datasheet" "" (id 3) (at 180.34 74.93 0)
+      (effects (font (size 1.27 1.27)) hide)
+    )
+    (pin "1")
+    (pin "2")
+    (pin "3")
+  )
+  (symbol (lib_id "Componentes proyecto:IRFP150") (at 124.46 73.66 0) (unit 1)
+    (in_bom yes) (on_board yes)
+    (property "Reference" "Q1" (id 0) (at 128.27 74.9299 0)
+      (effects (font (size 1.27 1.27)) (justify left))
+    )
+    (property "Value" "" (id 1) (at 128.27 77.4699 0)
+      (effects (font (size 1.27 1.27)) (justify left))
+    )
+    (property "Footprint" "" (id 2) (at 124.46 73.66 0)
+      (effects (font (size 1.27 1.27)) hide)
+    )
+    (property "Datasheet" "" (id 3) (at 124.46 73.66 0)
+      (effects (font (size 1.27 1.27)) hide)
+    )
+    (pin "1")
+    (pin "2")
+    (pin "3")
+  )
+  (symbol (lib_id "Componentes proyecto:IRFP150") (at 180.34 92.71 0) (unit 1)
+    (in_bom yes) (on_board yes) (fields_autoplaced)
+    (property "Reference" "Q4" (id 0) (at 184.15 92.7099 0)
+      (effects (font (size 1.27 1.27)) (justify left))
+    )
+    (property "Value" "" (id 1) (at 184.15 95.2499 0)
+      (effects (font (size 1.27 1.27)) (justify left))
+    )
+    (property "Footprint" "" (id 2) (at 180.34 92.71 0)
+      (effects (font (size 1.27 1.27)) hide)
+    )
+    (property "Datasheet" "" (id 3) (at 180.34 92.71 0)
+      (effects (font (size 1.27 1.27)) hide)
+    )
+    (pin "1")
+    (pin "2")
+    (pin "3")
+  )
   (sheet_instances
     (path "/" (page "1"))
   )
+  (symbol_instances
+    (path "/cb428b0a-31d9-482e-aaeb-be1bd1808598"
+      (reference "Q1") (unit 1) (value "IRFP150") (footprint "Package_TO_SOT_THT:TO-247-3_Horizontal_TabDown")
+    )
+    (path "/634b8e8d-237f-45e2-ab6d-e1f014df724a"
+      (reference "Q2") (unit 1) (value "IRFP150") (footprint "Package_TO_SOT_THT:TO-247-3_Horizontal_TabDown")
+    )
+    (path "/bd64a590-a69f-40d1-9a85-b87fef8d0c41"
+      (reference "Q3") (unit 1) (value "IRFP150") (footprint "Package_TO_SOT_THT:TO-247-3_Horizontal_TabDown")
+    )
+    (path "/de4f692d-4dfc-4a17-8571-883add49e290"
+      (reference "Q4") (unit 1) (value "IRFP150") (footprint "Package_TO_SOT_THT:TO-247-3_Horizontal_TabDown")
+    )
+    (path "/8dcf966e-c1a9-449b-a92c-2f0df5131b54"
+      (reference "U1") (unit 1) (value "UCC21540") (footprint "Package_SO:SOIC-16W_7.5x10.3mm_P1.27mm")
+    )
+    (path "/afd19999-467c-4454-a685-71d57851e5ed"
+      (reference "U2") (unit 1) (value "UCC21540") (footprint "Package_SO:SOIC-16W_7.5x10.3mm_P1.27mm")
+    )
+  )
 )
