File: Conversor/Proyecto-KiCAD/Proyecto-KiCAD.kicad_sch (KiCad schematic)
At the start: 43 parts, among them J2 ConnPila, J3 ConnTrafoP, J4 ConnTrafoS, J5 ConnLf, J6 ConnCarga, Q1 IRFP150, Q2 IRFP150, Q3 IRFP150, Q4 IRFP150, U1 ACPL-P480, U2 ACPL-P480, U3 ACPL-P480, U4 ACPL-P480, U5 2ED21834-S06J, U6 2ED21834-S06J

Commit message: Reestructurar el esquemático, con todo en heirarchical sheets
- Agregar la sheet de la placa adaptadora del DSP
Por hacer:
  - Completar la sheet del DSP con el proyecto de la placa adaptadora
Parts:
- removed C1: Csnub1, symbol Device:C_Small
- removed C10, C9: CDT, symbol Device:C_Small
- removed C11, C12: CVCC, symbol Device:C_Small
- removed C13, C14: Cboot, symbol Device:C_Small
- removed C15: CS, symbol Device:C_Small
- removed C16: Cin, symbol Device:C_Polarized_Small
- removed C17: Cf, symbol Device:C_Polarized
- removed C2: Csnub2, symbol Device:C_Small
- removed C3: Csnub3, symbol Device:C_Small
- removed C4: Csnub4, symbol Device:C_Small
- removed C5, C6, C7, C8: C, symbol Device:C_Small
- removed D1, D2, D3, D4: MUR860, Package_TO_SOT_THT:TO-220F-2_Vertical, symbol Componentes proyecto:MUR860
- removed J2: ConnPila, symbol Connector_Generic:Conn_01x02
- removed J3: ConnTrafoP, symbol Connector_Generic:Conn_01x02
- removed J4: ConnTrafoS, symbol Connector_Generic:Conn_01x02
- removed J5: ConnLf, symbol Connector_Generic:Conn_01x02
- removed J6: ConnCarga, symbol Connector_Generic:Conn_01x02
- removed Q1, Q2, Q3, Q4: IRFP150, Package_TO_SOT_THT:TO-247-3_Vertical, symbol Componentes proyecto:IRFP150
- removed R1, R3: RonH, symbol Device:R_US
- removed R2, R4: RonL, symbol Device:R_US
- removed R5, R6: RS, symbol Device:R_US
- removed R7: RS, symbol Device:R_Shunt_US
- removed U1, U2, U3, U4: ACPL-P480, Package_SO:SSO-6_6.8x4.6mm_P1.27mm_Clearance7mm, symbol Componentes proyecto:ACPL-P480
- removed U5: 2ED21834-S06J, symbol Componentes proyecto:2ED21834-S06J
- removed U6: 2ED21834-S06J, Package_SO:SOIC-14_3.9x8.7mm_P1.27mm, symbol Componentes proyecto:2ED21834-S06J
Other:
- added sheet Conversor (Conversor.kicad_sch)
- added sheet Drivers y Optos (DriversOptos.kicad_sch)
- added sheet Placa DSP (PlacaDSP.kicad_sch)
- sheet Fuentes ports: added +3.3V, +5VD, +5VP, VDDA; removed none
- sheet Sensores ports: added ALARMOUT, CLK, DATAIN, DATAOUT, IHALL+, IOUT, ISHUNT+, ISHUNT-, VIN, VOUT/IHALL-; removed none
- note added: "Alimentación digital"
- note added: "Alimentación potencia"
- note removed: "100nF"
- note removed: "10nF"
- note removed: "1uF"
- note removed: "200nF"
- note removed: "2Ω"
- note removed: "5.6Ω"
- note removed: "680 uF"
- note removed: "=4mΩ"
- note removed: "DT para proteccion de shoot-through (Evitar corto de una pata de MOSFETs)"
- note removed: "Io=(Vcc-1.2V)/((1.6//5)Ω+5.6Ω+1.5Ω)=1.06A"
- note removed: "RS para reducir picos negativos de VS"
- note removed: "tDT=400ns @ RDT=0Ω"
- note removed: "≈100nF"
- note removed: "≈15A f. de escala"
